File: pcb/Si5351BCBreakout.kicad_sch (KiCad schematic)
At the start: 49 parts, among them J1 Power/IO, J10 CLK2, J11 CLK4, J12 CLK0, J2 VC/CLKIN, J3 VC/CLKIN, J4 PS Sel, J5 3.3V Sel, J6 CLK3-CLK7, J7 CLK4, J8 CLK0, J9 CLK2, Q1 BSS138, Q2 BSS138, U1 LP2985-3.3, U2 ASTX-H11-25.000MHZ-T, U3 Si5351B/C

Commit message: Add missing 3d models, file cleanup
Parts:
- removed R17: 10k, Resistor_SMD:R_0805_2012Metric, symbol EtherkitKicadLibrary:R
Changed lines of the file:
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@@
 	(wire
 		(pts
-			(xy 219.71 138.43) (xy 215.9 138.43)
-		)
-		(stroke
-			(width 0)
-			(type default)
-		)
-	)
-	(wire
-		(pts
 			(xy 204.47 106.68) (xy 199.39 106.68)
 		)
@@
 		)
 	)
-	(global_label "VC_INTR"
-		(shape input)
-		(at 208.28 138.43 180)
-		(effects
-			(font
-				(size 1.27 1.27)
-			)
-			(justify right)
-		)
-		(property "Intersheetrefs" "${INTERSHEET_REFS}"
-			(at 208.28 138.43 0)
-			(hide yes)
-			(show_name no)
-			(do_not_autoplace no)
-			(effects
-				(font
-					(size 1.27 1.27)
-				)
-			)
-		)
-	)
 	(global_label "CLK7"
 		(shape input)
@@
 	(symbol
 		(lib_id "EtherkitKicadLibrary:R")
-		(at 212.09 138.43 270)
-		(unit 1)
-		(body_style 1)
-		(exclude_from_sim no)
-		(in_bom yes)
-		(on_board yes)
-		(in_pos_files yes)
-		(dnp no)
-		(property "Reference" "R17"
-			(at 212.09 133.985 90)
-			(show_name no)
-			(do_not_autoplace no)
-			(effects
-				(font
-					(size 1.27 1.27)
-				)
-			)
-		)
-		(property "Value" "10k"
-			(at 212.09 135.89 90)
-			(show_name no)
-			(do_not_autoplace no)
-			(effects
-				(font
-					(size 1.27 1.27)
-				)
-			)
-		)
-		(property "Footprint" "Resistor_SMD:R_0805_2012Metric"
-			(at 212.09 138.43 0)
-			(hide yes)
-			(show_name no)
-			(do_not_autoplace no)
-			(effects
-				(font
-					(size 1.524 1.524)
-				)
-			)
-		)
-		(property "Datasheet" ""
-			(at 212.09 138.43 0)
-			(show_name no)
-			(do_not_autoplace no)
-			(effects
-				(font
-					(size 1.524 1.524)
-				)
-			)
-		)
-		(property "Description" ""
-			(at 212.09 138.43 0)
-			(show_name no)
-			(do_not_autoplace no)
-			(effects
-				(font
-					(size 1.27 1.27)
-				)
-			)
-		)
-		(pin "1"
-		)
-		(pin "2"
-		)
-		(instances
-			(project "Si5351BCBreakout"
-				(path "/790cb86a-cab8-4bac-a34d-669b0923a386"
-					(reference "R17")
-					(unit 1)
-				)
-			)
-		)
-	)
-	(symbol
-		(lib_id "EtherkitKicadLibrary:R")
 		(at 212.09 146.05 270)
 		(unit 1)
@@
 					(unit 1)
 				)
-			)
-		)
-	)
-	(symbol
-		(lib_id "EtherkitKicadLibrary:+3.3VREG")
-		(at 219.71 138.43 0)
-		(unit 1)
-		(body_style 1)
-		(exclude_from_sim no)
-		(in_bom yes)
-		(on_board yes)
-		(in_pos_files yes)
-		(dnp no)
-		(property "Reference" "#PWR045"
-			(at 219.71 139.446 0)
-			(hide yes)
-			(show_name no)
-			(do_not_autoplace no)
-			(effects
-				(font
-					(size 0.762 0.762)
-				)
-			)
-		)
-		(property "Value" "+3.3VREG"
-			(at 219.9386 134.5438 0)
-			(show_name no)
-			(do_not_autoplace no)
-			(effects
-				(font
-					(size 1.27 1.27)
-				)
-			)
-		)
-		(property "Footprint" ""
-			(at 219.71 138.43 0)
-			(show_name no)
-			(do_not_autoplace no)
-			(effects
-				(font
-					(size 1.524 1.524)
-				)
-			)
-		)
-		(property "Datasheet" ""
-			(at 219.71 138.43 0)
-			(show_name no)
-			(do_not_autoplace no)
-			(effects
-				(font
-					(size 1.524 1.524)
-				)
-			)
-		)
-		(property "Description" ""
-			(at 219.71 138.43 0)
-			(show_name no)
-			(do_not_autoplace no)
-			(effects
-				(font
-					(size 1.27 1.27)
-				)
-			)
-		)
-		(pin "1"
-		)
-		(instances
-			(project "Si5351BCBreakout"
-				(path "/790cb86a-cab8-4bac-a34d-669b0923a386"
-					(reference "#PWR045")
-					(unit 1)
-				)

Commit message: TCXO change
Parts:
- removed R5, R8: 300, Resistor_SMD:R_0805_2012Metric, symbol EtherkitKicadLibrary:R
- removed R6: 18, Resistor_SMD:R_0805_2012Metric, symbol EtherkitKicadLibrary:R
- added C5: 100n, Capacitor_SMD:C_0805_2012Metric, symbol EtherkitKicadLibrary:C
- added R14, R15, R16: 0, Resistor_SMD:R_0805_2012Metric, symbol EtherkitKicadLibrary:R
- C1, C3: LCSC (none) -> C1779; MPN (none) -> CL21A475KAQNNNE; Manufacturer (none) -> Samsung Electro-Mechanics
- C10: renamed from C9; LCSC (none) -> C49678; MPN (none) -> CC0805KRX7R9BB104; Manufacturer (none) -> YAGEO
- C2: LCSC (none) -> C1710; MPN (none) -> CL21B103KBANNNC; Manufacturer (none) -> Samsung Electro-Mechanics
- C4: LCSC (none) -> C49678; MPN (none) -> CC0805KRX7R9BB104; Manufacturer (none) -> YAGEO
- C6: renamed from C5; LCSC (none) -> C49678; MPN (none) -> CC0805KRX7R9BB104; Manufacturer (none) -> YAGEO
- C7: renamed from C6; LCSC (none) -> C49678; MPN (none) -> CC0805KRX7R9BB104; Manufacturer (none) -> YAGEO
- C8: renamed from C7; LCSC (none) -> C49678; MPN (none) -> CC0805KRX7R9BB104; Manufacturer (none) -> YAGEO
- C9: renamed from C8; LCSC (none) -> C49678; MPN (none) -> CC0805KRX7R9BB104; Manufacturer (none) -> YAGEO
- H1, H4, J1, J10, J11, J12, J2, J3, J4, J5, J6, J7, J8, J9: now not fitted
- H2: renamed from H3; now not fitted
- H3: renamed from H2; now not fitted
- Q1, Q2: LCSC (none) -> C40912; MPN (none) -> BSS138-7-F; Manufacturer (none) -> Diodes Incorporated
- R1: renamed from R2; LCSC (none) -> C17414; MPN (none) -> 0805W8F1002T5E; Manufacturer (none) -> UNI-ROYAL(Uniroyal Elec)
- R10: renamed from R13; LCSC (none) -> C17415; MPN (none) -> 0805W8F100JT5E; Manufacturer (none) -> UNI-ROYAL(Uniroyal Elec)
- R11: renamed from R14; LCSC (none) -> C17415; MPN (none) -> 0805W8F100JT5E; Manufacturer (none) -> UNI-ROYAL(Uniroyal Elec)
- R12: renamed from R15; LCSC (none) -> C17415; MPN (none) -> 0805W8F100JT5E; Manufacturer (none) -> UNI-ROYAL(Uniroyal Elec)
- R13: renamed from R16; LCSC (none) -> C17415; MPN (none) -> 0805W8F100JT5E; Manufacturer (none) -> UNI-ROYAL(Uniroyal Elec)
- R17: renamed from R18; LCSC (none) -> C17414; MPN (none) -> 0805W8F1002T5E; Manufacturer (none) -> UNI-ROYAL(Uniroyal Elec)
- R18: renamed from R19; LCSC (none) -> C17414; MPN (none) -> 0805W8F1002T5E; Manufacturer (none) -> UNI-ROYAL(Uniroyal Elec)
- R2: renamed from R4; LCSC (none) -> C17414; MPN (none) -> 0805W8F1002T5E; Manufacturer (none) -> UNI-ROYAL(Uniroyal Elec)
- R3: renamed from R1; LCSC (none) -> C17477; MPN (none) -> 0805W8F0000T5E; Manufacturer (none) -> UNI-ROYAL(Uniroyal Elec); now not fitted
- R4: renamed from R3; LCSC (none) -> C17415; MPN (none) -> 0805W8F100JT5E; Manufacturer (none) -> UNI-ROYAL(Uniroyal Elec)
- R5: renamed from R7; LCSC (none) -> C17414; MPN (none) -> 0805W8F1002T5E; Manufacturer (none) -> UNI-ROYAL(Uniroyal Elec)
- R6: renamed from R9; LCSC (none) -> C17414; MPN (none) -> 0805W8F1002T5E; Manufacturer (none) -> UNI-ROYAL(Uniroyal Elec)
- R7: renamed from R10; LCSC (none) -> C17414; MPN (none) -> 0805W8F1002T5E; Manufacturer (none) -> UNI-ROYAL(Uniroyal Elec)
- R8: renamed from R11; LCSC (none) -> C17414; MPN (none) -> 0805W8F1002T5E; Manufacturer (none) -> UNI-ROYAL(Uniroyal Elec)
- R9: renamed from R12; LCSC (none) -> C17415; MPN (none) -> 0805W8F100JT5E; Manufacturer (none) -> UNI-ROYAL(Uniroyal Elec)
- U1: LCSC (none) -> C16085; MPN (none) -> LP2985AIM5-3.3/NOPB; Manufacturer (none) -> Texas Instruments
- U2: value ASTX-H11-25.000MHZ-T -> 25 MHz TCXO; LCSC (none) -> C48888230; MPN (none) -> OW2EL89CENUXK7YLC-25M; Manufacturer (none) -> YXC
- U3: Manufacturer (none) -> Skyworks
Connections:
- net CLK0: now also R15.2; no longer J12.1 (In), J8.1 (Pin_1)
- net CLK2: now also R16.2; no longer J10.1 (In), J9.1 (Pin_1)
- net CLK4: now also R14.2; no longer J11.1 (In), J7.1 (Pin_1)
- net at U3.1 (XA): now also C5.2
- net at R3.2, U2.1 (OE): no longer U3.2 (XB)
- net at U2.3 (OUT): now also C5.1
- new net CLK0_OUT: J12.1 (In), J8.1 (Pin_1), R15.1
- new net CLK2_OUT: J10.1 (In), J9.1 (Pin_1), R16.1
- new net CLK4_OUT: J11.1 (In), J7.1 (Pin_1), R14.1
- no-connect marks 0 -> 1
Other:
- moved on the sheet: C4, R4, U2

Commit message: Add logos to PCB
Changed lines of the file:
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@@
+		)
+	)
+	(symbol
+		(lib_id "Graphic:Logo_Open_Hardware_Small")
+		(at 191.77 59.69 0)
+		(unit 1)
+		(body_style 1)
+		(exclude_from_sim yes)
+		(in_bom no)
+		(on_board no)
+		(in_pos_files yes)
+		(dnp no)
+		(fields_autoplaced yes)
+		(property "Reference" "#SYM1"
+			(at 191.77 52.705 0)
+			(hide yes)
+			(show_name no)
+			(do_not_autoplace no)
+			(effects
+				(font
+					(size 1.27 1.27)
+				)
+			)
+		)
+		(property "Value" "Logo_Open_Hardware_Small"
+			(at 191.77 65.405 0)
+			(hide yes)
+			(show_name no)
+			(do_not_autoplace no)
+			(effects
+				(font
+					(size 1.27 1.27)
+				)
+			)
+		)
+		(property "Footprint" "Symbol:OSHW-Symbol_6.7x6mm_SilkScreen"
+			(at 191.77 59.69 0)
+			(hide yes)
+			(show_name no)
+			(do_not_autoplace no)
+			(effects
+				(font
+					(size 1.27 1.27)
+				)
+			)
+		)
+		(property "Datasheet" ""
+			(at 191.77 59.69 0)
+			(hide yes)
+			(show_name no)
+			(do_not_autoplace no)
+			(effects
+				(font
+					(size 1.27 1.27)
+				)
+			)
+		)
+		(property "Description" "Open Hardware logo, small"
+			(at 191.77 59.69 0)
+			(hide yes)
+			(show_name no)
+			(do_not_autoplace no)
+			(effects
+				(font
+					(size 1.27 1.27)
+				)
+			)
+		)
+		(instances
+			(project "Si5351BCBreakout"
+				(path "/790cb86a-cab8-4bac-a34d-669b0923a386"
+					(reference "#SYM1")
+					(unit 1)
+				)
+			)
+		)
+	)
+	(symbol
+		(lib_id "Etherkit KiCad Library:LOGO")
+		(at 213.36 58.42 0)
+		(unit 1)
+		(body_style 1)
+		(exclude_from_sim no)
+		(in_bom yes)
+		(on_board yes)
+		(in_pos_files yes)
+		(dnp no)
+		(fields_autoplaced yes)
+		(property "Reference" "#G1"
+			(at 213.36 54.055 0)
+			(hide yes)
+			(show_name no)
+			(do_not_autoplace no)
+			(effects
+				(font
+					(size 1.27 1.27)
+				)
+			)
+		)
+		(property "Value" "LOGO"
+			(at 213.36 62.785 0)
+			(hide yes)
+			(show_name no)
+			(do_not_autoplace no)
+			(effects
+				(font
+					(size 1.27 1.27)
+				)
+			)
+		)
+		(property "Footprint" "Etherkit KiCad Library:EtherkitLogoSmall"
+			(at 213.36 58.42 0)
+			(hide yes)
+			(show_name no)
+			(do_not_autoplace no)
+			(effects
+				(font
+					(size 1.27 1.27)
+				)
+			)
+		)
+		(property "Datasheet" ""
+			(at 213.36 58.42 0)
+			(hide yes)
+			(show_name no)
+			(do_not_autoplace no)
+			(effects
+				(font
+					(size 1.27 1.27)
+				)
+			)
+		)
+		(property "Description" ""
+			(at 213.36 58.42 0)
+			(hide yes)
+			(show_name no)
+			(do_not_autoplace no)
+			(effects
+				(font
+					(size 1.27 1.27)
+				)
+			)
+		)
+		(instances
+			(project "Si5351BCBreakout"
+				(path "/790cb86a-cab8-4bac-a34d-669b0923a386"
+					(reference "#G1")
+					(unit 1)
+				)
+			)
 		)
 	)
